Commit message: Add files via upload

File: robot_omni/urdf/omni_base.urdf (robot description, URDF)
Before this commit: robot omni_base, 17 links, 16 joints
Links:
- added link base_rgbd_camera_bottom_screw_frame
- added link base_rgbd_camera_link, mass 0.072; collision box size=0.02505 0.09 0.025; visual mesh filename=file:///opt/ros/jazzy/share/realsense2_description/meshes/d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
- added link cameras_add_on_link, mass 3.057; collision mesh filename=file:///home/nahhao74/ros2_ws/install/omni_base_description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 scale=1 1 1; visual mesh filename=file:///home/nahhao74/ros2_ws/install/omni_base_description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 scale=1 1 1
- added link roof_rgbd_camera_bottom_screw_frame
- added link roof_rgbd_camera_link, mass 0.072; collision box size=0.02505 0.09 0.025; visual mesh filename=file:///opt/ros/jazzy/share/realsense2_description/meshes/d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
Joints:
- added joint base_rgbd_camera_joint: type fixed, parent base_link, child base_rgbd_camera_bottom_screw_frame, origin xyz=0.327327              0.0              0.551436 rpy=0.0             0.0             0.0
- added joint base_rgbd_camera_link_joint: type fixed, parent base_rgbd_camera_bottom_screw_frame, child base_rgbd_camera_link, origin xyz=0.010600000000000002 0.0175 0.0125 rpy=0 0 0
- added joint cameras_add_on_joint: type fixed, parent base_link, child cameras_add_on_link, origin xyz=0.0 0.0 0.0 rpy=0 0 0, axis 0 0 1
- added joint roof_rgbd_camera_joint: type fixed, parent base_link, child roof_rgbd_camera_bottom_screw_frame, origin xyz=0.297329              0.0              0.483197 rpy=0.0              0.20943951023931956              0.0
- added joint roof_rgbd_camera_link_joint: type fixed, parent roof_rgbd_camera_bottom_screw_frame, child roof_rgbd_camera_link, origin xyz=0.010600000000000002 0.0175 0.0125 rpy=0 0 0
